Commit message: updated dual urdf file

File: daurar_description/urdf/dual_arm_setup.urdf (robot description, URDF)
Before this commit: robot ur5, 40 links, 39 joints
Joints:
- joint left_shoulder_lift_joint: origin xyz=0.0 0.13585 0.0 rpy=0.0 1.57079632679 0.0 -> xyz=0.0 0.13585 0.0 rpy=0.0 -1.57079632679 0.0
- joint left_shoulder_pan_joint: origin xyz=0.0 0.0 0.089159 rpy=0.0 0.0 0.0 -> xyz=0.0 0.0 0.089159 rpy=0 0 3.14159265359
- joint left_wrist_1_joint: origin xyz=0.0 0.0 0.39225 rpy=0.0 1.57079632679 0.0 -> xyz=0.0 0.0 0.39225 rpy=0.0 -1.57079632679 0.0
- joint left_wrist_2_joint: origin xyz=0.0 0.093 0.0 rpy=0.0 0.0 0.0 -> xyz=0.0 0.093 0.0 rpy=0 0 0
- joint left_wrist_3_joint: origin xyz=0.0 0.0 0.09465 rpy=0.0 0.0 0.0 -> xyz=0.0 0.0 0.09465 rpy=0 0 0
- joint world_joint_1: origin xyz=0.645 0.635 1.275 rpy=0.0 2.35619449019  0.0 -> xyz=0.645 0.635 1.275 rpy=-2.35619 0 -1.57079632679
