Commit message: Added ur5_right_arm configuration

File: daurar_description/urdf/right_arm_setup.urdf (robot description, URDF)
Before this commit: robot ur5, 40 links, 39 joints
Links:
- removed link left_base
- removed link left_base_link
- removed link left_ee_link
- removed link left_forearm_link
- removed link left_gripper_base_link
- removed link left_gripper_finger1_finger_link
- removed link left_gripper_finger1_finger_tip_link
- removed link left_gripper_finger1_inner_knuckle_link
- removed link left_gripper_finger1_knuckle_link
- removed link left_gripper_finger2_finger_link
- removed link left_gripper_finger2_finger_tip_link
- removed link left_gripper_finger2_inner_knuckle_link
- removed link left_gripper_finger2_knuckle_link
- removed link left_shoulder_link
- removed link left_tool0
- removed link left_upper_arm_link
- removed link left_wrist_1_link
- removed link left_wrist_2_link
- removed link left_wrist_3_link
Joints:
- removed joint left_base_link-base_fixed_joint
- removed joint left_ee_fixed_joint
- removed joint left_elbow_joint
- removed joint left_gripper_base_joint
- removed joint left_gripper_finger1_finger_joint
- removed joint left_gripper_finger1_finger_tip_joint
- removed joint left_gripper_finger1_inner_knuckle_joint
- removed joint left_gripper_finger1_joint
- removed joint left_gripper_finger2_finger_joint
- removed joint left_gripper_finger2_finger_tip_joint
- removed joint left_gripper_finger2_inner_knuckle_joint
- removed joint left_gripper_finger2_joint
- removed joint left_shoulder_lift_joint
- removed joint left_shoulder_pan_joint
- removed joint left_wrist_1_joint
- removed joint left_wrist_2_joint
- removed joint left_wrist_3_joint
- removed joint left_wrist_3_link-tool0_fixed_joint
- removed joint world_joint_1
